File: Shift_registers.kicad_sch (KiCad schematic)
At the start: 24 parts, among them J5 Conn_01x10_Socket, K1 G3MB-202P, K2 G3MB-202P, K3 G3MB-202P, K4 G3MB-202P, K5 G3MB-202P, K6 G3MB-202P, K7 G3MB-202P, K8 G3MB-202P, K9 G3MB-202P, U3 ULN2803A, U4 74HC595D_118, U5 ULN2803A, U6 74HC595D_118

Commit message: Almoust done
Parts:
- renumbered J5 to J6, R15 to R14, U3 to U4, U4 to U5, U5 to U6, U6 to U7
Changed lines of the file:
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@@
 		(dnp no)
 		(fields_autoplaced yes)
-		(property "Reference" "U3"
+		(property "Reference" "U4"
 			(at 154.94 52.07 0)
 			(show_name no)
@@
 			(project "WachcioDrop"
 				(path "/cc2cb50c-70f7-486a-b07b-c403b0b67709/e2e3bbe9-9850-463c-a6b0-6dd792bf3c12"
-					(reference "U3")
+					(reference "U4")
 					(unit 1)
 				)
@@
 		(in_pos_files yes)
 		(dnp no)
-		(property "Reference" "U6"
+		(property "Reference" "U7"
 			(at 65.786 188.976 0)
 			(show_name no)
@@
 			(project "WachcioDrop"
 				(path "/cc2cb50c-70f7-486a-b07b-c403b0b67709/e2e3bbe9-9850-463c-a6b0-6dd792bf3c12"
-					(reference "U6")
+					(reference "U7")
 					(unit 1)
 				)
@@
 		(dnp no)
 		(fields_autoplaced yes)
-		(property "Reference" "#PWR030"
+		(property "Reference" "#PWR032"
 			(at 22.86 80.01 0)
 			(hide yes)
@@
 			(project "WachcioDrop"
 				(path "/cc2cb50c-70f7-486a-b07b-c403b0b67709/e2e3bbe9-9850-463c-a6b0-6dd792bf3c12"
-					(reference "#PWR030")
+					(reference "#PWR032")
 					(unit 1)
 				)
@@
 		(in_pos_files yes)
 		(dnp no)
-		(property "Reference" "#PWR025"
+		(property "Reference" "#PWR027"
 			(at 232.41 50.8 0)
 			(hide yes)
@@
 			(project "WachcioDrop"
 				(path "/cc2cb50c-70f7-486a-b07b-c403b0b67709/e2e3bbe9-9850-463c-a6b0-6dd792bf3c12"
-					(reference "#PWR025")
+					(reference "#PWR027")
 					(unit 1)
 				)
@@
 		(dnp no)
 		(fields_autoplaced yes)
-		(property "Reference" "#PWR038"
+		(property "Reference" "#PWR040"
 			(at 116.84 167.64 0)
 			(hide yes)
@@
 			(project "WachcioDrop"
 				(path "/cc2cb50c-70f7-486a-b07b-c403b0b67709/e2e3bbe9-9850-463c-a6b0-6dd792bf3c12"
-					(reference "#PWR038")
+					(reference "#PWR040")
 					(unit 1)
 				)
@@
 		(dnp no)
 		(fields_autoplaced yes)
-		(property "Reference" "J5"
+		(property "Reference" "J6"
 			(at 161.29 189.23 90)
 			(show_name no)
@@
 			(project "WachcioDrop"
 				(path "/cc2cb50c-70f7-486a-b07b-c403b0b67709/e2e3bbe9-9850-463c-a6b0-6dd792bf3c12"
-					(reference "J5")
+					(reference "J6")
 					(unit 1)
 				)
@@
 		(dnp no)
 		(fields_autoplaced yes)
-		(property "Reference" "#PWR036"
+		(property "Reference" "#PWR038"
 			(at 24.13 144.78 0)
 			(hide yes)
@@
 			(project "WachcioDrop"
 				(path "/cc2cb50c-70f7-486a-b07b-c403b0b67709/e2e3bbe9-9850-463c-a6b0-6dd792bf3c12"
-					(reference "#PWR036")
+					(reference "#PWR038")
 					(unit 1)
 				)
@@
 		(in_pos_files yes)
 		(dnp no)
-		(property "Reference" "#PWR035"
+		(property "Reference" "#PWR037"
 			(at 130.81 130.81 0)
 			(hide yes)
@@
 			(project "WachcioDrop"
 				(path "/cc2cb50c-70f7-486a-b07b-c403b0b67709/e2e3bbe9-9850-463c-a6b0-6dd792bf3c12"
-					(reference "#PWR035")
+					(reference "#PWR037")
 					(unit 1)
 				)
@@
 		(in_pos_files yes)
 		(dnp no)
-		(property "Reference" "R15"
+		(property "Reference" "R14"
 			(at 92.202 148.59 90)
 			(show_name no)
@@
 			(project "WachcioDrop"
 				(path "/cc2cb50c-70f7-486a-b07b-c403b0b67709/e2e3bbe9-9850-463c-a6b0-6dd792bf3c12"
-					(reference "R15")
+					(reference "R14")
 					(unit 1)
 				)
@@
 		(dnp no)
 		(fields_autoplaced yes)
-		(property "Reference" "#PWR031"
+		(property "Reference" "#PWR033"
 			(at 19.05 80.01 0)
 			(hide yes)
@@
 			(project "WachcioDrop"
 				(path "/cc2cb50c-70f7-486a-b07b-c403b0b67709/e2e3bbe9-9850-463c-a6b0-6dd792bf3c12"
-					(reference "#PWR031")
+					(reference "#PWR033")
 					(unit 1)
 				)
@@
 		(dnp no)
 		(fields_autoplaced yes)
-		(property "Reference" "#PWR027"
+		(property "Reference" "#PWR029"
 			(at 22.86 54.61 0)
 			(hide yes)
@@
 			(project "WachcioDrop"
 				(path "/cc2cb50c-70f7-486a-b07b-c403b0b67709/e2e3bbe9-9850-463c-a6b0-6dd792bf3c12"
-					(reference "#PWR027")
+					(reference "#PWR029")
 					(unit 1)
 				)
@@
 		(dnp no)
 		(fields_autoplaced yes)
-		(property "Reference" "#PWR032"
+		(property "Reference" "#PWR034"
 			(at 154.94 95.25 0)
 			(hide yes)
@@
 			(project "WachcioDrop"
 				(path "/cc2cb50c-70f7-486a-b07b-c403b0b67709/e2e3bbe9-9850-463c-a6b0-6dd792bf3c12"
-					(reference "#PWR032")
+					(reference "#PWR034")
 					(unit 1)
 				)
@@
 		(in_pos_files yes)
 		(dnp no)
-		(property "Reference" "#PWR022"
+		(property "Reference" "#PWR024"
 			(at 180.34 25.4 0)
 			(hide yes)
@@
 			(project "WachcioDrop"
 				(path "/cc2cb50c-70f7-486a-b07b-c403b0b67709/e2e3bbe9-9850-463c-a6b0-6dd792bf3c12"
-					(reference "#PWR022")
+					(reference "#PWR024")
 					(unit 1)
 				)
@@
 		(dnp no)
 		(fields_autoplaced yes)
-		(property "Reference" "#PWR040"
+		(property "Reference" "#PWR042"
 			(at 38.1 190.5 0)
 			(hide yes)
@@
 			(project "WachcioDrop"
 				(path "/cc2cb50c-70f7-486a-b07b-c403b0b67709/e2e3bbe9-9850-463c-a6b0-6dd792bf3c12"
-					(reference "#PWR040")
+					(reference "#PWR042")
 					(unit 1)
 				)
@@
 		(in_pos_files yes)
 		(dnp no)
-		(property "Reference" "#PWR024"
+		(property "Reference" "#PWR026"
 			(at 184.15 50.8 0)
 			(hide yes)
@@
 			(project "WachcioDrop"
 				(path "/cc2cb50c-70f7-486a-b07b-c403b0b67709/e2e3bbe9-9850-463c-a6b0-6dd792bf3c12"
-					(reference "#PWR024")
+					(reference "#PWR026")
 					(unit 1)
 				)
@@
 		(dnp no)
 		(fields_autoplaced yes)
-		(property "Reference" "U5"
+		(property "Reference" "U6"
 			(at 116.84 123.19 0)
 			(show_name no)
@@
 			(project "WachcioDrop"
 				(path "/cc2cb50c-70f7-486a-b07b-c403b0b67709/e2e3bbe9-9850-463c-a6b0-6dd792bf3c12"
-					(reference "U5")
+					(reference "U6")
 					(unit 1)
 				)
@@
 		(dnp no)
 		(fields_autoplaced yes)
-		(property "Reference" "#PWR039"
+		(property "Reference" "#PWR041"
 			(at 20.32 170.18 0)
 			(hide yes)
@@
 			(project "WachcioDrop"
 				(path "/cc2cb50c-70f7-486a-b07b-c403b0b67709/e2e3bbe9-9850-463c-a6b0-6dd792bf3c12"
-					(reference "#PWR039")
+					(reference "#PWR041")
 					(unit 1)
 				)
@@
 		(in_pos_files yes)
 		(dnp no)
-		(property "Reference" "#PWR034"
+		(property "Reference" "#PWR036"
 			(at 232.41 104.14 0)
 			(hide yes)
@@
 			(project "WachcioDrop"
 				(path "/cc2cb50c-70f7-486a-b07b-c403b0b67709/e2e3bbe9-9850-463c-a6b0-6dd792bf3c12"
-					(reference "#PWR034")
+					(reference "#PWR036")
 					(unit 1)
 				)
@@
 		(in_pos_files yes)
 		(dnp no)
-		(property "Reference" "#PWR026"
+		(property "Reference" "#PWR028"
 			(at 168.91 59.69 0)
 			(hide yes)
@@
 			(project "WachcioDrop"
 				(path "/cc2cb50c-70f7-486a-b07b-c403b0b67709/e2e3bbe9-9850-463c-a6b0-6dd792bf3c12"
-					(reference "#PWR026")
+					(reference "#PWR028")
 					(unit 1)
 				)
@@
 		(in_pos_files yes)
 		(dnp no)
-		(property "Reference" "#PWR028"
+		(property "Reference" "#PWR030"
 			(at 189.23 76.2 0)
 			(hide yes)
@@
 			(project "WachcioDrop"
 				(path "/cc2cb50c-70f7-486a-b07b-c403b0b67709/e2e3bbe9-9850-463c-a6b0-6dd792bf3c12"
-					(reference "#PWR028")
+					(reference "#PWR030")
 					(unit 1)
 				)
@@
 		(in_pos_files yes)
 		(dnp no)
-		(property "Reference" "#PWR033"
+		(property "Reference" "#PWR035"
 			(at 189.23 104.14 0)
 			(hide yes)
@@
 			(project "WachcioDrop"
 				(path "/cc2cb50c-70f7-486a-b07b-c403b0b67709/e2e3bbe9-9850-463c-a6b0-6dd792bf3c12"
-					(reference "#PWR033")
+					(reference "#PWR035")
 					(unit 1)
 				)
@@
 		(in_pos_files yes)
 		(dnp no)
-		(property "Reference" "U4"
+		(property "Reference" "U5"
 			(at 60.198 100.33 0)
 			(show_name no)
@@
 			(project "WachcioDrop"
 				(path "/cc2cb50c-70f7-486a-b07b-c403b0b67709/e2e3bbe9-9850-463c-a6b0-6dd792bf3c12"
-					(reference "U4")
+					(reference "U5")
 					(unit 1)
 				)
@@
 		(in_pos_files yes)
 		(dnp no)
-		(property "Reference" "#PWR029"
+		(property "Reference" "#PWR031"
 			(at 232.41 76.2 0)
 			(hide yes)
@@
 			(project "WachcioDrop"
 				(path "/cc2cb50c-70f7-486a-b07b-c403b0b67709/e2e3bbe9-9850-463c-a6b0-6dd792bf3c12"
-					(reference "#PWR029")
+					(reference "#PWR031")
 					(unit 1)
 				)
@@
 		(in_pos_files yes)
 		(dnp no)
-		(property "Reference" "#PWR037"
+		(property "Reference" "#PWR039"
 			(at 144.78 154.94 0)
 			(hide yes)
@@
 			(project "WachcioDrop"
 				(path "/cc2cb50c-70f7-486a-b07b-c403b0b67709/e2e3bbe9-9850-463c-a6b0-6dd792bf3c12"
-					(reference "#PWR037")
+					(reference "#PWR039")
 					(unit 1)
 				)
@@
 		(in_pos_files yes)
 		(dnp no)
-		(property "Reference" "#PWR023"
+		(property "Reference" "#PWR025"
 			(at 229.87 26.67 0)
 			(hide yes)
@@
 			(project "WachcioDrop"
 				(path "/cc2cb50c-70f7-486a-b07b-c403b0b67709/e2e3bbe9-9850-463c-a6b0-6dd792bf3c12"
-					(reference "#PWR023")
+					(reference "#PWR025")
 					(unit 1)
 				)
