File: WachcioDrop.kicad_sch (KiCad schematic)
At the start: 23 parts, among them J1 Conn_02x20_Top_Bottom, J2 Conn_01x04, J3 Conn_01x03, J4 Screw_Terminal_01x02, U1 TC00500 RTC DS3231, U2 ESP32-S3-DEVKITC-1-N8R2, U7 LM1117RS-3.3

Commit message: Almoust done
Parts:
- added J4: Conn_01x03, Connector_PinHeader_2.54mm:PinHeader_1x03_P2.54mm_Vertical, symbol symbols:Conn_01x03
- C1: value C_Polarized -> 800uF 50V
- renumbered J4 to J5, U7 to U3
Connections:
- net +3.3V: now also J4.1 (Pin_1)
- net GND: now also J4.3 (Pin_3)
- net PIN_DS18B20: now also J4.2 (Pin_2)
Other:
- moved on the sheet: J2
