File: display_board.kicad_pcb (KiCad board)
At the start: 4 copper layers, 100 x 100 mm, 23 parts, among them J7 Conn_02x20_Top_Bottom

Commit message: Fix some errors after build PCBs
Changed lines of the file:
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@@
 		(tags "LED")
 		(property "Reference" "D13"
-			(at 1.27 -3 0)
+			(at 3.04 -2.175 0)
 			(unlocked yes)
 			(layer "F.SilkS")
@@
 		)
 		(property "Value" "LED"
-			(at 1.27 2.06 0)
+			(at 2.605714 2.06 0)
 			(unlocked yes)
 			(layer "F.Fab")
@@
 		)
 		(property "Value" "LED"
-			(at 1.27 2.06 0)
+			(at 2.671429 2 0)
 			(unlocked yes)
 			(layer "F.Fab")
@@
 		)
 		(property "Value" "LED"
-			(at 1.27 2.06 0)
+			(at 2.802857 2.06 0)
 			(unlocked yes)
 			(layer "F.Fab")
@@
 		)
 		(property "Value" "LED"
-			(at 1.27 2.06 0)
+			(at 2.737143 2.06 0)
 			(unlocked yes)
 			(layer "F.Fab")
@@
 		)
 		(property "Value" "LED"
-			(at 1.27 2.06 0)
+			(at 3.5 2.06 0)
 			(unlocked yes)
 			(layer "F.Fab")
@@
 		)
 		(property "Value" "LED"
-			(at 1.27 2.06 0)
+			(at 2.54 2.06 0)
 			(unlocked yes)
 			(layer "F.Fab")
@@
 		(tags "LED")
 		(property "Reference" "D14"
-			(at 3.04 -3 0)
+			(at 3.04 -2.175 0)
 			(unlocked yes)
 			(layer "F.SilkS")
@@
 		)
 		(property "Value" "LED"
-			(at -0.96 -3 0)
+			(at -1.46 -2.175 0)
 			(unlocked yes)
 			(layer "F.Fab")
@@
 		)
 		(property "Value" "LED"
-			(at 1.27 2.06 0)
+			(at 2.77 2.06 0)
 			(unlocked yes)
 			(layer "F.Fab")
@@
 		)
 		(property "Value" "LED"
-			(at 1.27 2.06 0)
+			(at 2.934286 2.06 0)
 			(unlocked yes)
 			(layer "F.Fab")
@@
 		)
 		(property "Value" "LED"
-			(at 1.27 2.06 0)
+			(at 2.868571 2.06 0)
 			(unlocked yes)
 			(layer "F.Fab")
@@
 		)
 	)
+	(gr_poly
+		(pts
+			(xy 106 81.5) (xy 106 83.5) (xy 104.5 82.5)
+		)
+		(stroke
+			(width 0.1)
+			(type solid)
+		)
+		(fill yes)
+		(layer "F.SilkS")
+	)
+	(gr_poly
+		(pts
+			(xy 106.356412 74.929059) (xy 106.356412 76.929059) (xy 104.856412 75.929059)
+		)
+		(stroke
+			(width 0.1)
+			(type solid)
+		)
+		(fill yes)
+		(layer "F.SilkS")
+	)
+	(gr_poly
+		(pts
+			(xy 114 75) (xy 114 77) (xy 112.5 76)
+		)
+		(stroke
+			(width 0.1)
+			(type solid)
+		)
+		(fill yes)
+		(layer "F.SilkS")
+	)
+	(gr_poly
+		(pts
+			(xy 122 75) (xy 122 77) (xy 120.5 76)
+		)
+		(stroke
+			(width 0.1)
+			(type solid)
+		)
+		(fill yes)
+		(layer "F.SilkS")
+	)
+	(gr_poly
+		(pts
+			(xy 130 75) (xy 130 77) (xy 128.5 76)
+		)
+		(stroke
+			(width 0.1)
+			(type solid)
+		)
+		(fill yes)
+		(layer "F.SilkS")
+	)
+	(gr_poly
+		(pts
+			(xy 138 75) (xy 138 77) (xy 136.5 76)
+		)
+		(stroke
+			(width 0.1)
+			(type solid)
+		)
+		(fill yes)
+		(layer "F.SilkS")
+	)
+	(gr_poly
+		(pts
+			(xy 146 75) (xy 146 77) (xy 144.5 76)
+		)
+		(stroke
+			(width 0.1)
+			(type solid)
+		)
+		(fill yes)
+		(layer "F.SilkS")
+	)
+	(gr_poly
+		(pts
+			(xy 154 75) (xy 154 77) (xy 152.5 76)
+		)
+		(stroke
+			(width 0.1)
+			(type solid)
+		)
+		(fill yes)
+		(layer "F.SilkS")
+	)
+	(gr_poly
+		(pts
+			(xy 162 75) (xy 162 77) (xy 160.5 76)
+		)
+		(stroke
+			(width 0.1)
+			(type solid)
+		)
+		(fill yes)
+		(layer "F.SilkS")
+	)
+	(gr_poly
+		(pts
+			(xy 184 21.5) (xy 184 23.5) (xy 182.5 22.5)
+		)
+		(stroke
+			(width 0.1)
+			(type solid)
+		)
+		(fill yes)
+		(layer "F.SilkS")
+	)
+	(gr_poly
+		(pts
+			(xy 193 21.5) (xy 193 23.5) (xy 191.5 22.5)
+		)
+		(stroke
+			(width 0.1)
+			(type solid)
+		)
+		(fill yes)
+		(layer "F.SilkS")
+	)
 	(gr_line
