File: main_board.kicad_pcb (KiCad board)
At the start: 4 copper layers, 100 x 100 mm, 51 parts, among them J1 Conn_02x20_Top_Bottom, J2 Conn_01x04, J3 Conn_01x03, J4 Conn_01x03, J5 Screw_Terminal_01x02, J6 Conn_01x10_Socket, K1 G3MB-202P, K2 G3MB-202P, K3 G3MB-202P, K4 G3MB-202P, K5 G3MB-202P, K6 G3MB-202P, K7 G3MB-202P, K8 G3MB-202P, K9 G3MB-202P, U1 TC00500 RTC DS3231, U2 ESP32-S3-DEVKITC-1-N8R2, U3 LM1117RS-3.3, U4 ULN2803A, U5 74HC595D_118, U6 ULN2803A, U7 74HC595D_118

Commit message: Add GND in PS1. Flip PS1
Parts:
- PS1: moved to B.Cu
- moved PS1 1.10 mm to (171.5, 104.8)
Routing:
- net GND: track 46.7 -> 54.2 mm
- net +5V: track 142.6 -> 138.2 mm
- net Net-(D1-+): track 13.4 -> 11.5 mm

Commit message: Fix some errors after build PCBs
Parts:
- PS1: moved to F.Cu
- moved PS1 1.75 mm to (171.5, 106.5), turned to 0 degrees
Routing:
- net GND: track 54.2 -> 71.9 mm
- net Net-(D1-+): track 11.5 -> 19.9 mm
- net +5V: track 138.2 -> 138.9 mm
